File: Dille.kicad_sch (KiCad schematic)
At the start: 69 parts, among them Q1 MMBFJ112, SW2 SW_DPDT_x2, U1 PT2399, U2 TL074, U3 L78L05_SOT89

Commit message: pcb
Parts:
- added J1: Barrel_Jack_Switch, Connector_BarrelJack:BarrelJack_Kycon_KLDX-0202-xC_Horizontal, symbol Connector:Barrel_Jack_Switch
- C14, C19, C21, C25: footprint Capacitor_SMD:CP_Elec_4x5.4 -> Capacitor_SMD:CP_Elec_4x4.5; LCSC# C4747969 -> C249787
- C2, C20: footprint Capacitor_SMD:CP_Elec_6.3x5.4 -> Capacitor_SMD:CP_Elec_6.3x4.5; LCSC# C37308 -> C5374787
- TP1: value 9V IN -> GND; footprint TestPoint:TestPoint_THTPad_D2.5mm_Drill1.2mm -> TestPoint:Test point 2.5x1.5
- TP2, TP3, TP4: footprint TestPoint:TestPoint_THTPad_D2.5mm_Drill1.2mm -> TestPoint:Test point 2.5x1.5
- renumbered R3 to R11, R5 to R13, R7 to R14, R11 to R3, R13 to R5, R14 to R7
Connections:
- net GND: now also TP1.1, J1.1
- net at R1.1: now also J1.2; no longer TP1.1
- no-connect marks 4 -> 5
Other:
- moved on the sheet: C5, D1, R1, R2, R4, TP4

Commit message: pcb 2
Connections:
- net Sig in: now reaches C6.1, R6.1, TP2.1
- net Sig out: now reaches C25.2, R23.1, TP3.1
Changed lines of the file:
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@@
     (effects (font (size 2.54 2.54) (thickness 0.508) bold) (justify left bottom))
+  )
+  (global_label "Sig in" (shape input) (at 25.4 43.18 0) (fields_autoplaced)
+    (effects (font (size 1.27 1.27)) (justify left))
+    (property "Intersheetrefs" "${INTERSHEET_REFS}" (at 33.9905 43.18 0)
+      (effects (font (size 1.27 1.27)) (justify left) hide)
+    )
   )
   (global_label "+4V5" (shape input) (at 40.64 26.67 0) (fields_autoplaced)
@@
       (effects (font (size 1.27 1.27)) (justify right) hide)
     )
+  )
+  (global_label "Sig out" (shape input) (at 166.37 76.2 180) (fields_autoplaced)
+    (effects (font (size 1.27 1.27)) (justify right))
+    (property "Intersheetrefs" "${INTERSHEET_REFS}" (at 156.5096 76.2 0)
+      (effects (font (size 1.27 1.27)) (justify right) hide)
+    )

Commit message: Rev 2
Parts:
- C1, C10, C11, C12, C13, C14, C15, C16, C17, C18, C19, C2, C20, C21, C22, C23, C24, C25, C26, C3, C4, C5, C6, C7, C8, C9, D1, D2, Q1, R1, R10, R11, R12, R13, R14, R15, R16, R17, R18, R19, R2, R20, R21, R22, R23, R24, R25, R26, R27, R3, R4, R5, R6, R7, R8, R9, U1, U2, U3: supplier (none) -> LCSC

Commit message: Silkscreen updated
Parts:
- added TP5, TP6: TestPoint, TestPoint:TestPoint_Pad_4.0x4.0mm, symbol Connector:TestPoint
Connections:
- net GND: now also TP6.1
- net at J1.2, R1.1: now also TP5.1
Changed lines of the file:
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@@
   (junction (at 119.38 128.27) (diameter 0) (color 0 0 0 0)
   )
+  (junction (at 203.2 45.72) (diameter 0) (color 0 0 0 0)
+  )
   (junction (at 210.82 27.94) (diameter 0) (color 0 0 0 0)
   )
@@
   (junction (at 245.11 78.74) (diameter 0) (color 0 0 0 0)
   )
+  (junction (at 200.66 27.94) (diameter 0) (color 0 0 0 0)
+  )
   (junction (at 80.01 80.01) (diameter 0) (color 0 0 0 0)
   )
@@
     (stroke (width 0) (type default))
   )
+  (wire (pts (xy 200.66 27.94) (xy 203.2 27.94))
+    (stroke (width 0) (type default))
+  )
   (wire (pts (xy 82.55 124.46) (xy 82.55 128.27))
     (stroke (width 0) (type default))
@@
     (stroke (width 0) (type default))
   )
-  (wire (pts (xy 198.12 27.94) (xy 203.2 27.94))
+  (wire (pts (xy 198.12 27.94) (xy 200.66 27.94))
     (stroke (width 0) (type default))
   )
@@
     (stroke (width 0) (type default))
   )
+  (wire (pts (xy 203.2 45.72) (xy 210.82 45.72))
+    (stroke (width 0) (type default))
+  )
   (wire (pts (xy 240.03 27.94) (xy 240.03 36.83))
     (stroke (width 0) (type default))
@@
     (stroke (width 0) (type default))
   )
+  (wire (pts (xy 200.66 25.4) (xy 200.66 27.94))
+    (stroke (width 0) (type default))
+  )
   (wire (pts (xy 33.02 128.27) (xy 35.56 128.27))
     (stroke (width 0) (type default))
@@
     (stroke (width 0) (type default))
   )
-  (wire (pts (xy 200.66 45.72) (xy 210.82 45.72))
+  (wire (pts (xy 200.66 45.72) (xy 203.2 45.72))
     (stroke (width 0) (type default))
   )
@@
         )
       )
+    )
+  )
+  (symbol (lib_id "Connector:TestPoint") (at 203.2 45.72 180) (unit 1)
+    (in_bom yes) (on_board yes) (dnp no)
+    (property "Reference" "TP6" (at 205.74 49.657 0)
+      (effects (font (size 1.27 1.27)) (justify right))
+    )
+    (property "Value" "TestPoint" (at 205.74 47.117 0)
+      (effects (font (size 1.27 1.27)) (justify right))
+    )
+    (property "Footprint" "TestPoint:TestPoint_Pad_4.0x4.0mm" (at 198.12 45.72 0)
+      (effects (font (size 1.27 1.27)) hide)
+    )
+    (property "Datasheet" "~" (at 198.12 45.72 0)
+      (effects (font (size 1.27 1.27)) hide)
+    )
+    (pin "1")
+    (instances
+      (project "Dille"
+        (path "/641bcc8c-dd98-40c2-a746-7885ee720607"
+          (reference "TP6") (unit 1)
+        )
+      )
+    )
+  )
+  (symbol (lib_id "Connector:TestPoint") (at 200.66 25.4 0) (unit 1)
+    (in_bom yes) (on_board yes) (dnp no)
+    (property "Reference" "TP5" (at 198.12 21.463 0)
+      (effects (font (size 1.27 1.27)) (justify right))
+    )
+    (property "Value" "TestPoint" (at 198.12 24.003 0)
+      (effects (font (size 1.27 1.27)) (justify right))
+    )
+    (property "Footprint" "TestPoint:TestPoint_Pad_4.0x4.0mm" (at 205.74 25.4 0)
+      (effects (font (size 1.27 1.27)) hide)
+    )
+    (property "Datasheet" "~" (at 205.74 25.4 0)
+      (effects (font (size 1.27 1.27)) hide)
+    )
+    (pin "1")
+    (instances
+      (project "Dille"
+        (path "/641bcc8c-dd98-40c2-a746-7885ee720607"
+          (reference "TP5") (unit 1)
+        )
+      )

Commit message: Revision 2
Parts:
- removed R24, R25, R26, R27: 100k, Resistor_SMD:R_0805_2012Metric_Pad1.20x1.40mm_HandSolder, symbol Device:R_Small
- removed U2: TL074, Package_SO:SO-14_3.9x8.65mm_P1.27mm, symbol Amplifier_Operational:TL074
- added U4: TL072, Package_SO:SO-8_3.9x4.9mm_P1.27mm, symbol Amplifier_Operational:TL072
Connections:
- net +4V5: now also U4.5 (+)
- net +9V: now also U4.8 (V+)
- net GND: now also U4.4 (V-)
- net at Q1.1 (D), R13.2: now also U4.1, U4.2 (-)
- net at R11.2: now also U4.3 (+)
- net at C24.1, R21.1, R8.1: now also U4.7
- net at C24.2, R13.1, R20.1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: now also U4.6 (-)
